Commit message: feat/refactor_URDF_read

File: SO-ARM101-OMNI-KIN.urdf (robot description, URDF)
Before this commit: robot SO-ARM101-OMNI-KIN, 9 links, 8 joints
Links:
- added link gripper_tcp
Joints:
- added joint gripper_tcp_joint: type fixed, parent gripper_base, child gripper_tcp, origin xyz=0 0.0369151517 0.0369152807 rpy=2.356194490192345 0 3.141592653589793
